File: ESP32_RTC.kicad_pcb (KiCad board)
At the start: 2 copper layers, 43.5 x 54 mm, 40 parts, among them J1 Screw_Terminal_01x02, J3 Conn_01x04_Pin, SW1 SW_Push, SW2 SW_Push, U1 DS3231M, U2 MAX7219, U3 ESP32-WROOM-32, U4 CC56-12SRWA, U5 AMS1117

Commit message: image update
Parts:
- moved C6 34.7 mm to (105.1, 99.7)
- moved D1 34.7 mm to (107.0, 89.3)
- moved D3 34.7 mm to (117.1, 89.6)
- moved H1 34.7 mm to (106.4, 112.5)
- moved H4 34.7 mm to (106.3, 71.0)
- moved R4 34.7 mm to (118.4, 105.4)
- moved R6 34.7 mm to (105.1, 92.0)
- moved REF** 34.7 mm to (123.7, 74.4)
- moved SW1 34.7 mm to (107.9, 82.1)
- moved C3 34.7 mm to (130.1, 109.2)
- moved C4 34.7 mm to (130.1, 111.4)
- moved C5 34.7 mm to (105.1, 97.6)
- moved C7 34.7 mm to (110.8, 72.2)
- moved D2 34.7 mm to (112.5, 87.3)
- moved H2 34.7 mm to (143.1, 112.5)
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Routing:
- net GND: track 233.4 -> 243.7 mm
Other:
- outline, holes or cut-outs redrawn
