File: ESP32_RTC.kicad_sch (KiCad schematic)
At the start: 37 parts, among them J1 Screw_Terminal_01x02, J3 Conn_01x04_Pin, SW1 SW_Push, SW2 SW_Push, U1 DS3231M, U2 MAX7219, U3 ESP32-WROOM-32, U4 CC56-12SRWA, U5 AMS1117

Commit message: image update
Changed lines of the file:
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@@
 					(size 1.27 1.27)
 				)
-				(hide yes)
 			)
 		)
